Commit message: Rename motion_execution to snp_motion_execution and update rosinstall

File: ros2_ws/src/snp_support/urdf/workcell.xacro (robot description, xacro)
@@ -26,8 +26,22 @@
     </collision>
   </link>
+  <link name="camera_link"/>
+  <link name="target_base_link"/>
   <joint name="tool0_to_pushcorp_base" type="fixed">
     <parent link="tool0"/>
     <child link="pushcorp_base"/>
     <origin xyz="0 0 0.01635" rpy="${pi/2} 0 ${pi}"/>
+    <axis xyz="0 0 0"/>
+  </joint>
+  <joint name="robot_to_camera_joint" type="fixed">
+    <parent link="tool0"/>
+    <child link="camera_link"/>
+    <origin xyz="0 0 0" rpy="0 0 0"/>
+    <axis xyz="0 0 0"/>
+  </joint>
+  <joint name="world_to_target_joint" type="fixed">
+    <parent link="floor"/>
+    <child link="target_base_link"/>
+    <origin xyz="0.7 0 0.15" rpy="0 0 -${pi/2}"/>
     <axis xyz="0 0 0"/>
   </joint>

Commit message: Add deps_ws

File: ros2_ws/src/snp_support/urdf/workcell.xacro (robot description, xacro)
@@ -27,5 +27,11 @@
   </link>
   <link name="camera_link"/>
-  <link name="target_base_link"/>
+  <link name="target_base_link">
+    <visual>
+      <geometry>
+        <mesh filename="package://snp_support/meshes/rosWorldCalib.dae"/>
+      </geometry>
+    </visual>
+  </link>
   <joint name="tool0_to_pushcorp_base" type="fixed">
     <parent link="tool0"/>

Commit message: Clean launching of systems

File: ros2_ws/src/snp_support/urdf/workcell.xacro (robot description, xacro)
@@ -29,4 +29,5 @@
   <link name="target_base_link">
     <visual>
+      <origin xyz="0.37565 0.2809875 0" rpy="${pi/2} 0 ${pi}"/>
       <geometry>
         <mesh filename="package://snp_support/meshes/rosWorldCalib.dae"/>
@@ -49,5 +50,5 @@
     <parent link="floor"/>
     <child link="target_base_link"/>
-    <origin xyz="0.7 0 0.15" rpy="0 0 -${pi/2}"/>
+    <origin xyz="0.555 0.061 0.126" rpy="0.004 -0.004 -1.628"/>
     <axis xyz="0 0 0"/>
   </joint>

Commit message: Additional testing changes

File: ros2_ws/src/snp_support/urdf/workcell.xacro (robot description, xacro)
@@ -52,4 +52,16 @@
     <origin xyz="0.555 0.061 0.126" rpy="0.004 -0.004 -1.628"/>
     <axis xyz="0 0 0"/>
+  </joint>
+  <link name="camera_color_optical_frame"/>
+  <link name="target_cal_frame"/>
+  <joint name="camera_cal_joint" type="fixed">
+    <parent link="camera_link"/>
+    <child link="camera_color_optical_frame"/>
+    <origin xyz="0.085549560652492 -0.1732631672558103 0.1329373703855808" wxyz="0.5118596229748543 -0.5074314040915237 0.4900425218487801 -0.4902768843111336"/>
+  </joint>
+  <joint name="target_cal_joint" type="fixed">
+    <parent link="floor"/>
+    <child link="target_cal_frame"/>
+    <origin xyz="0.555641489380775 0.05956001933889868 0.1229851433910979" wxyz="0.6869783604862724 -0.001114251051880176 -0.003909064875724348 -0.7266665052690842"/>
   </joint>
   <!-- TODO do we care about effort and velocity limits?-->

Commit message: Most recent changes

File: ros2_ws/src/snp_support/urdf/workcell.xacro (robot description, xacro)
@@ -2,4 +2,10 @@
 <robot name="snp_workcell" xmlns:xacro="http://ros.org/wiki/xacro">
   <xacro:include filename="$(find snp_support)/urdf/mh180_120.xacro"/>
+  <material name="light_gray">
+    <color rgba="0.7 0.7 0.7 1"/>
+  </material>
+  <material name="dark_gray">
+    <color rgba="0.3 0.3 0.3 1"/>
+  </material>
   <link name="pushcorp_base">
     <visual>
@@ -16,11 +22,14 @@
   <link name="pushcorp_compliance">
     <visual>
-      <geometry>
-        <mesh filename="package://snp_support/meshes/pushcorp/pushcorp_compliance.dae"/>
-      </geometry>
-    </visual>
-    <collision>
-      <geometry>
-        <mesh filename="package://snp_support/meshes/pushcorp/pushcorp_compliance.dae"/>
+      <origin xyz="0 0.059 0" rpy="${pi} 0 0"/>
+      <geometry>
+        <mesh filename="package://snp_support/meshes/pushcorp/pushcorp_spindle.dae"/>
+      </geometry>
+      <material name="light_gray"/>
+    </visual>
+    <collision>
+      <origin xyz="0 0.059 0" rpy="${pi} 0 0"/>
+      <geometry>
+        <mesh filename="package://snp_support/meshes/pushcorp/pushcorp_spindle.dae"/>
       </geometry>
     </collision>
@@ -38,6 +47,5 @@
     <parent link="tool0"/>
     <child link="pushcorp_base"/>
-    <origin xyz="0 0 0.01635" rpy="${pi/2} 0 ${pi}"/>
-    <axis xyz="0 0 0"/>
+    <origin xyz="0 0 0.01635" rpy="${pi/2} 0 0"/>
   </joint>
   <joint name="robot_to_camera_joint" type="fixed">
@@ -73,13 +81,7 @@
     <limit upper="0.01778" lower="-0.01778" effort="0" velocity="0"/>
   </joint>
-  <material name="light_gray">
-    <color rgba="0.7 0.7 0.7 1"/>
-  </material>
-  <material name="dark_gray">
-    <color rgba="0.3 0.3 0.3 1"/>
-  </material>
   <xacro:property name="platform_height" value="${5*0.0254}"/>
-  <xacro:property name="mount_height" value="${19.6*0.0254}"/>
-  <xacro:property name="mount_width" value="${28.5*0.0254}"/>
+  <xacro:property name="robot_mount_height" value="${19.6*0.0254}"/>
+  <xacro:property name="robot_mount_width" value="${28.5*0.0254}"/>
   <xacro:property name="pushcorp_box_height" value="${30*0.0254}"/>
   <xacro:property name="pushcorp_box_width" value="${17*0.0254}"/>
@@ -88,4 +90,7 @@
   <xacro:property name="control_boxes_width" value="${38*0.0254}"/>
   <xacro:property name="control_boxes_length" value="${130*0.0254}"/>
+  <xacro:property name="table_height" value="${33.875*0.0254}"/>
+  <xacro:property name="table_width" value="${48*0.0254}"/>
+  <xacro:property name="table_length" value="${30*0.0254}"/>
   <link name="floor"/>
   <link name="platform">
@@ -105,11 +110,11 @@
     <visual>
       <geometry>
-        <box size="${mount_width} ${mount_width} ${mount_height}"/>
-      </geometry>
-      <material name="dark_gray"/>
-    </visual>
-    <collision>
-      <geometry>
-        <box size="${mount_width} ${mount_width} ${mount_height}"/>
+        <box size="${robot_mount_width} ${robot_mount_width} ${robot_mount_height}"/>
+      </geometry>
+      <material name="dark_gray"/>
+    </visual>
+    <collision>
+      <geometry>
+        <box size="${robot_mount_width} ${robot_mount_width} ${robot_mount_height}"/>
       </geometry>
     </collision>
@@ -167,15 +172,19 @@
     </collision>
   </link>
+  <link name="buffy_tcp"/>
+  <joint name="buffy_tcp_joint" type="fixed">
+    <parent link="tool0"/>
+    <child link="buffy_tcp"/>
+    <origin xyz="0.292 0 0.19" rpy="0 -${pi/2} 0"/>
+  </joint>
   <joint name="floor_to_platform" type="fixed">
     <parent link="floor"/>
     <child link="platform"/>
     <origin xyz="0 0 ${platform_height/2}" rpy="0 0 0"/>
-    <axis xyz="0 0 0"/>
   </joint>
   <joint name="platform_to_mount" type="fixed">
     <parent link="platform"/>
     <child link="robot_mount"/>
-    <origin xyz="0 0 ${platform_height/2 + mount_height/2}" rpy="0 0 0"/>
-    <axis xyz="0 0 0"/>
+    <origin xyz="0 0 ${platform_height/2 + robot_mount_height/2}" rpy="0 0 0"/>
   </joint>
   <joint name="floor_to_control_boxes" type="fixed">
@@ -183,29 +192,24 @@
     <child link="control_boxes"/>
     <origin xyz="${4*0.0254 + control_boxes_length/2} -${56*0.0254 + control_boxes_width/2} ${control_boxes_height/2}" rpy="0 0 0"/>
-    <axis xyz="0 0 0"/>
   </joint>
   <joint name="mount_to_base" type="fixed">
     <parent link="robot_mount"/>
     <child link="base_link"/>
-    <origin xyz="0 0 ${mount_height/2}" rpy="0 0 0"/>
-    <axis xyz="0 0 0"/>
+    <origin xyz="0 0 ${robot_mount_height/2}" rpy="0 0 0"/>
   </joint>
   <joint name="floor_to_pushcorp_support_1" type="fixed">
     <parent link="floor"/>
     <child link="pushcorp_box_support_1"/>
-    <origin xyz="-${mount_width/2 + 2.75*0.0254} ${mount_width/2 + 16.25*0.0254} ${20.25*0.0254+platform_height}" rpy="0 0 0"/>
-    <axis xyz="0 0 0"/>
+    <origin xyz="-${robot_mount_width/2 + 2.75*0.0254} ${robot_mount_width/2 + 16.25*0.0254} ${20.25*0.0254+platform_height}" rpy="0 0 0"/>
   </joint>
   <joint name="floor_to_pushcorp_support_2" type="fixed">
     <parent link="floor"/>
     <child link="pushcorp_box_support_2"/>
-    <origin xyz="-${mount_width/2 + 1.25*0.0254 + pushcorp_box_length} ${mount_width/2 + 16.25*0.0254} ${20.25*0.0254+platform_height}" rpy="0 0 0"/>
-    <axis xyz="0 0 0"/>
+    <origin xyz="-${robot_mount_width/2 + 1.25*0.0254 + pushcorp_box_length} ${robot_mount_width/2 + 16.25*0.0254} ${20.25*0.0254+platform_height}" rpy="0 0 0"/>
   </joint>
   <joint name="floor_to_pushcorp_box" type="fixed">
     <parent link="floor"/>
     <child link="pushcorp_box"/>
-    <origin xyz="-${mount_width/2 + 2*0.0254 + pushcorp_box_length/2} ${mount_width/2 + 17*0.0254 + pushcorp_box_width/2} ${14*0.0254 + pushcorp_box_height/2}" rpy="0 0 0"/>
-    <axis xyz="0 0 0"/>
+    <origin xyz="-${robot_mount_width/2 + 2*0.0254 + pushcorp_box_length/2} ${robot_mount_width/2 + 17*0.0254 + pushcorp_box_width/2} ${14*0.0254 + pushcorp_box_height/2}" rpy="0 0 0"/>
   </joint>
 </robot>
