Commit message: update snp_support with new robot and end effector

File: snp_support/urdf/workcell.xacro (robot description, xacro)
@@ -1,5 +1,7 @@
 <?xml version="1.0" ?>
-<robot name="snp_workcell" xmlns:xacro="http://ros.org/wiki/xacro">
-  <xacro:include filename="$(find snp_support)/urdf/mh180_120.xacro"/>
+<robot name="motoman_hc10" xmlns:xacro="http://ros.org/wiki/xacro">
+  <xacro:include filename="$(find motoman_hc10_support)/urdf/hc10_macro.xacro" />
+  <xacro:motoman_hc10 prefix=""/>
+  <!-- Add World -->
   <material name="light_gray">
     <color rgba="0.7 0.7 0.7 1"/>
@@ -8,13 +10,61 @@
     <color rgba="0.3 0.3 0.3 1"/>
   </material>
+  <link name="world"/>
+  <!-- Add Floor -->
+  <xacro:property name="length" value="9.0"/>
+  <xacro:property name="width" value="6.0"/>
+  <link name="floor">
+    <visual>
+      <origin xyz="0 -${width/10} 0.001" rpy="0 0 0"/>
+      <geometry>
+        <box size="${length} ${width} 0.001"/>
+      </geometry>
+      <material name="tesseract_white"/>
+    </visual>
+    <collision>
+      <origin xyz="0 -${width/10} 0.001" rpy="0 0 0"/>
+      <geometry>
+        <box size="${length} ${width} 0.001"/>
+      </geometry>
+    </collision>
+  </link>
+  <joint name="world_to_floor" type="fixed">
+    <origin xyz="0 0 0" rpy="0 0 0"/>
+    <parent link="world"/>
+    <child link="floor"/>
+  </joint>
+  <!-- Add table -->
+  <link name="table">
+    <visual>
+      <geometry>
+        <mesh filename="package://snp_support/meshes/collision_demo/Steel Table 4 ft x 6ft.STL"/>
+      </geometry>
+      <material name="dark_gray"/>
+    </visual>
+    <collision>
+      <geometry>
+        <mesh filename="package://snp_support/meshes/collision_demo/convex_hulls/steel_table.ply"/>
+      </geometry>
+    </collision>
+  </link>
+  <joint name="floor_to_table" type="fixed">
+    <parent link="floor"/>
+    <child link="table"/>
+  </joint>
+  <joint name="table_to_base" type="fixed">
+    <parent link="table"/>
+    <child link="base_link"/>
+    <origin xyz="-0.61 0 0.723" rpy="0 0 0"/> <!-- model doesn't perfectly match .sldprt lenghts -->
+  </joint>
+  <!-- Add End Effector Components -->
   <link name="pushcorp_base">
     <visual>
       <geometry>
-        <mesh filename="package://snp_support/meshes/pushcorp/pushcorp_base.dae"/>
-      </geometry>
-    </visual>
-    <collision>
-      <geometry>
-        <mesh filename="package://snp_support/meshes/pushcorp/pushcorp_base.dae"/>
+        <mesh filename="package://snp_support/meshes/collision_demo/convex_hulls/afd310.ply"/>
+      </geometry>
+    </visual>
+    <collision>
+      <geometry>
+        <mesh filename="package://snp_support/meshes/collision_demo/convex_hulls/afd310.ply"/>
       </geometry>
     </collision>
@@ -22,21 +72,131 @@
   <link name="pushcorp_compliance">
     <visual>
-      <origin xyz="0 0.059 0" rpy="${pi} 0 0"/>
-      <geometry>
-        <mesh filename="package://snp_support/meshes/pushcorp/pushcorp_spindle.dae"/>
+      <geometry>
+        <mesh filename="package://snp_support/meshes/collision_demo/rps100.ply"/>
       </geometry>
       <material name="light_gray"/>
     </visual>
     <collision>
-      <origin xyz="0 0.059 0" rpy="${pi} 0 0"/>
-      <geometry>
-        <mesh filename="package://snp_support/meshes/pushcorp/pushcorp_spindle.dae"/>
-      </geometry>
-    </collision>
-  </link>
+      <geometry>
+        <mesh filename="package://snp_support/meshes/collision_demo/convex_hulls/rps100.ply"/>
+      </geometry>
+    </collision>
+  </link>
+  <link name="pushcorp_backplate">
+    <visual>
+      <geometry>
+        <mesh filename="package://snp_support/meshes/collision_demo/backplate.ply"/>
+      </geometry>
+    </visual>
+    <collision>
+      <geometry>
+        <mesh filename="package://snp_support/meshes/collision_demo/convex_hulls/backplate.ply"/>
+      </geometry>
+    </collision>
+  </link>
+  <joint name="tool0_to_pushcorp_backplate" type="fixed">
+    <parent link="tool0"/>
+    <child link="pushcorp_backplate"/>
+    <origin xyz="0 0 0" rpy="0 0 ${radians(180)}"/>
+  </joint>
+  <link name="pushcorp_camera1">
+    <visual>
+      <geometry>
+        <mesh filename="package://snp_support/meshes/collision_demo/camera1.ply"/>
+      </geometry>
+    </visual>
+    <collision>
+      <geometry>
+        <mesh filename="package://snp_support/meshes/collision_demo/convex_hulls/camera1.ply"/>
+      </geometry>
+    </collision>
+  </link>
+  <joint name="tool0_to_pushcorp_camera1" type="fixed">
+    <parent link="tool0"/>
+    <child link="pushcorp_camera1"/>
+    <origin xyz="0 0 0" rpy="0 0 ${radians(180)}"/>
+  </joint>
+  <link name="pushcorp_camera2">
+    <visual>
+      <geometry>
+        <mesh filename="package://snp_support/meshes/collision_demo/camera2.ply"/>
+      </geometry>
+    </visual>
+    <collision>
+      <geometry>
+        <mesh filename="package://snp_support/meshes/collision_demo/convex_hulls/camera2.ply"/>
+      </geometry>
+    </collision>
+  </link>
+  <joint name="tool0_to_pushcorp_camera2" type="fixed">
+    <parent link="tool0"/>
+    <child link="pushcorp_camera2"/>
+    <origin xyz="0 0 0" rpy="0 0 ${radians(180)}"/>
+  </joint>
+  <link name="pushcorp_frontplate">
+    <visual>
+      <geometry>
+        <mesh filename="package://snp_support/meshes/collision_demo/frontplate.ply"/>
+      </geometry>
+    </visual>
+    <collision>
+      <geometry>
+        <mesh filename="package://snp_support/meshes/collision_demo/convex_hulls/front.ply"/>
+      </geometry>
+    </collision>
+  </link>
+  <joint name="tool0_to_pushcorp_frontplate" type="fixed">
+    <parent link="tool0"/>
+    <child link="pushcorp_frontplate"/>
+    <origin xyz="0 0 0" rpy="0 0 ${radians(180)}"/>
+  </joint>
+  <joint name="tool0_to_pushcorp_base" type="fixed">
+    <parent link="tool0"/>
+    <child link="pushcorp_base"/>
+    <origin xyz="0 0 0" rpy="0 0 ${radians(180)}"/>
+  </joint>
+  <link name="pushcorp_sidebracket1">
+    <visual>
+      <geometry>
+        <mesh filename="package://snp_support/meshes/collision_demo/sidebracket1.ply"/>
+      </geometry>
+    </visual>
+    <collision>
+      <geometry>
+        <mesh filename="package://snp_support/meshes/collision_demo/convex_hulls/bracket1.ply"/>
+      </geometry>
+    </collision>
+  </link>
+  <joint name="tool0_to_pushcorp_sidebracket1" type="fixed">
+    <parent link="tool0"/>
+    <child link="pushcorp_sidebracket1"/>
+    <origin xyz="0 0 0" rpy="0 0 ${radians(180)}"/>
+  </joint>
+  <link name="pushcorp_sidebracket2">
+    <visual>
+      <geometry>
+        <mesh filename="package://snp_support/meshes/collision_demo/sidebracket2.ply"/>
+      </geometry>
+    </visual>
+    <collision>
+      <geometry>
+        <mesh filename="package://snp_support/meshes/collision_demo/convex_hulls/bracket2.ply"/>
+      </geometry>
+    </collision>
+  </link>
+  <joint name="tool0_to_pushcorp_sidebracket2" type="fixed">
+    <parent link="tool0"/>
+    <child link="pushcorp_sidebracket2"/>
+    <origin xyz="0 0 0" rpy="0 0 ${radians(180)}"/>
+  </joint>
+  <joint name="tool0_to_pushcorp_actuator" type="fixed">
+    <parent link="tool0"/>
+    <child link="pushcorp_compliance"/>
+    <origin xyz="0 0 0" rpy="0 0 ${radians(180)}"/>
+  </joint>
   <link name="camera_link"/>
+  <!-- Add Target Calibration -->
   <link name="target_base_link">
     <visual>
-      <origin xyz="0.37565 0.2809875 0" rpy="${pi/2} 0 ${pi}"/>
       <geometry>
         <mesh filename="package://snp_support/meshes/rosWorldCalib.dae"/>
@@ -44,20 +204,13 @@
     </visual>
   </link>
-  <joint name="tool0_to_pushcorp_base" type="fixed">
-    <parent link="tool0"/>
-    <child link="pushcorp_base"/>
-    <origin xyz="0 0 0.01635" rpy="${pi/2} 0 0"/>
-  </joint>
   <joint name="robot_to_camera_joint" type="fixed">
     <parent link="tool0"/>
     <child link="camera_link"/>
-    <origin xyz="0 0 0" rpy="0 0 0"/>
-    <axis xyz="0 0 0"/>
+    <origin xyz="0.175 0 0" rpy="0 0 0"/>
   </joint>
   <joint name="world_to_target_joint" type="fixed">
     <parent link="floor"/>
     <child link="target_base_link"/>
-    <origin xyz="0.555 0.061 0.126" rpy="0.004 -0.004 -1.628"/>
-    <axis xyz="0 0 0"/>
+    <origin xyz="0.37565 0.2809875 0.723" rpy="${pi/2} 0 ${pi}"/>
   </joint>
   <link name="camera_color_optical_frame"/>
@@ -66,150 +219,16 @@
     <parent link="camera_link"/>
     <child link="camera_color_optical_frame"/>
-    <origin xyz="0.085549560652492 -0.1732631672558103 0.1329373703855808" wxyz="0.5118596229748543 -0.5074314040915237 0.4900425218487801 -0.4902768843111336"/>
   </joint>
   <joint name="target_cal_joint" type="fixed">
     <parent link="floor"/>
     <child link="target_cal_frame"/>
-    <origin xyz="0.555641489380775 0.05956001933889868 0.1229851433910979" wxyz="0.6869783604862724 -0.001114251051880176 -0.003909064875724348 -0.7266665052690842"/>
-  </joint>
-  <!-- TODO do we care about effort and velocity limits?-->
-  <joint name="pushcorp_actuator" type="prismatic">
-    <parent link="pushcorp_base"/>
-    <child link="pushcorp_compliance"/>
-    <origin xyz="0 0 0" rpy="0 0 0"/>
-    <axis xyz="-1 0 0"/>
-    <limit upper="0.01778" lower="-0.01778" effort="0" velocity="0"/>
-  </joint>
-  <xacro:property name="platform_height" value="${5*0.0254}"/>
-  <xacro:property name="robot_mount_height" value="${19.6*0.0254}"/>
-  <xacro:property name="robot_mount_width" value="${28.5*0.0254}"/>
-  <xacro:property name="pushcorp_box_height" value="${30*0.0254}"/>
-  <xacro:property name="pushcorp_box_width" value="${17*0.0254}"/>
-  <xacro:property name="pushcorp_box_length" value="${28*0.0254}"/>
-  <xacro:property name="control_boxes_height" value="${60*0.0254}"/>
-  <xacro:property name="control_boxes_width" value="${38*0.0254}"/>
-  <xacro:property name="control_boxes_length" value="${130*0.0254}"/>
-  <xacro:property name="table_height" value="${33.875*0.0254}"/>
-  <xacro:property name="table_width" value="${48*0.0254}"/>
-  <xacro:property name="table_length" value="${30*0.0254}"/>
-  <link name="floor"/>
-  <link name="platform">
-    <visual>
-      <geometry>
-        <box size="${96*0.0254} ${72*0.0254} ${platform_height}"/>
-      </geometry>
-      <material name="dark_gray"/>
-    </visual>
-    <collision>
-      <geometry>
-        <box size="${96*0.0254} ${72*0.0254} ${platform_height}"/>
-      </geometry>
-    </collision>
-  </link>
-  <link name="robot_mount">
-    <visual>
-      <geometry>
-        <box size="${robot_mount_width} ${robot_mount_width} ${robot_mount_height}"/>
-      </geometry>
-      <material name="dark_gray"/>
-    </visual>
-    <collision>
-      <geometry>
-        <box size="${robot_mount_width} ${robot_mount_width} ${robot_mount_height}"/>
-      </geometry>
-    </collision>
-  </link>
-  <link name="pushcorp_box_support_1">
-    <visual>
-      <geometry>
-        <box size="${1.5*0.0254} ${1.5*0.0254} ${40.5*0.0254}" />
-      </geometry>
-      <material name="dark_gray"/>
-    </visual>
-    <collision>
-      <geometry>
-        <box size="${1.5*0.0254} ${1.5*0.0254} ${40.5*0.0254}" />
-      </geometry>
-    </collision>
-  </link>
-  <link name="pushcorp_box_support_2">
-    <visual>
-      <geometry>
-        <box size="${1.5*0.0254} ${1.5*0.0254} ${40.5*0.0254}" />
-      </geometry>
-      <material name="dark_gray"/>
-    </visual>
-    <collision>
-      <geometry>
-        <box size="${1.5*0.0254} ${1.5*0.0254} ${40.5*0.0254}" />
-      </geometry>
-    </collision>
-  </link>
-  <link name="pushcorp_box">
-    <visual>
-      <geometry>
-        <box size="${pushcorp_box_length} ${pushcorp_box_width} ${pushcorp_box_height}"/>
-      </geometry>
-      <material name="light_gray"/>
-    </visual>
-    <collision>
-      <geometry>
-        <box size="${pushcorp_box_length} ${pushcorp_box_width} ${pushcorp_box_height}"/>
-      </geometry>
-    </collision>
-  </link>
-  <link name="control_boxes">
-   <visual>
-      <geometry>
-        <box size="${control_boxes_length} ${control_boxes_width} ${control_boxes_height}"/>
-      </geometry>
-      <material name="light_gray"/>
-    </visual>
-    <collision>
-      <geometry>
-        <box size="${control_boxes_length} ${control_boxes_width} ${control_boxes_height}"/>
-      </geometry>
-    </collision>
-  </link>
-  <link name="buffy_tcp"/>
-  <joint name="buffy_tcp_joint" type="fixed">
-    <parent link="tool0"/>
-    <child link="buffy_tcp"/>
-    <origin xyz="0.292 0 0.19" rpy="0 -${pi/2} 0"/>
-  </joint>
-  <joint name="floor_to_platform" type="fixed">
-    <parent link="floor"/>
-    <child link="platform"/>
-    <origin xyz="0 0 ${platform_height/2}" rpy="0 0 0"/>
-  </joint>
-  <joint name="platform_to_mount" type="fixed">
-    <parent link="platform"/>
-    <child link="robot_mount"/>
-    <origin xyz="0 0 ${platform_height/2 + robot_mount_height/2}" rpy="0 0 0"/>
-  </joint>
-  <joint name="floor_to_control_boxes" type="fixed">
-    <parent link="floor"/>
-    <child link="control_boxes"/>
-    <origin xyz="${4*0.0254 + control_boxes_length/2} -${56*0.0254 + control_boxes_width/2} ${control_boxes_height/2}" rpy="0 0 0"/>
-  </joint>
-  <joint name="mount_to_base" type="fixed">
-    <parent link="robot_mount"/>
-    <child link="base_link"/>
-    <origin xyz="0 0 ${robot_mount_height/2}" rpy="0 0 0"/>
-  </joint>
-  <joint name="floor_to_pushcorp_support_1" type="fixed">
-    <parent link="floor"/>
-    <child link="pushcorp_box_support_1"/>
-    <origin xyz="-${robot_mount_width/2 + 2.75*0.0254} ${robot_mount_width/2 + 16.25*0.0254} ${20.25*0.0254+platform_height}" rpy="0 0 0"/>
-  </joint>
-  <joint name="floor_to_pushcorp_support_2" type="fixed">
-    <parent link="floor"/>
-    <child link="pushcorp_box_support_2"/>
-    <origin xyz="-${robot_mount_width/2 + 1.25*0.0254 + pushcorp_box_length} ${robot_mount_width/2 + 16.25*0.0254} ${20.25*0.0254+platform_height}" rpy="0 0 0"/>
-  </joint>
-  <joint name="floor_to_pushcorp_box" type="fixed">
-    <parent link="floor"/>
-    <child link="pushcorp_box"/>
-    <origin xyz="-${robot_mount_width/2 + 2*0.0254 + pushcorp_box_length/2} ${robot_mount_width/2 + 17*0.0254 + pushcorp_box_width/2} ${14*0.0254 + pushcorp_box_height/2}" rpy="0 0 0"/>
+    <origin xyz="0.37565 0.2809875 0.723" rpy="${pi/2} 0 ${pi}"/>
+  </joint>
+  <!-- Add TCP -->
+  <link name="sand_tcp"/>
+  <joint name="sand_tcp_joint" type="fixed">
+    <parent link="tool0"/>
+    <child link="sand_tcp"/>
+    <origin xyz="0.23261 0 0.08259" rpy="${radians(90)} 0 ${radians(90)}"/> <!-- values from solidworks -->
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
Commit message: Remove non-existent material

File: snp_support/urdf/workcell.xacro (robot description, xacro)
@@ -20,5 +20,4 @@
         <box size="${length} ${width} 0.001"/>
       </geometry>
-      <material name="tesseract_white"/>
     </visual>
     <collision>
