Commit message: Move MH180 meshes to MH180 directory

File: snp_blending/urdf/mh180_120/mh180_120_macro.xacro (robot description, xacro)
@@ -7,5 +7,5 @@
         <origin xyz="0 0 0" rpy="0 0 0"/>
         <geometry>
-          <mesh filename="package://snp_blending/meshes/mh180/visual/base_link.stl"/>
+          <mesh filename="package://snp_blending/urdf/mh180_120/visual/base_link.stl"/>
         </geometry>
         <material name="blue">
@@ -15,5 +15,5 @@
       <collision>
         <geometry>
-          <mesh filename="package://snp_blending/meshes/mh180/collision/base_link.stl"/>
+          <mesh filename="package://snp_blending/urdf/mh180_120/collision/base_link.stl"/>
         </geometry>
         <material name="yellow">
@@ -26,5 +26,5 @@
         <origin xyz="0 0 0" rpy="0 0 0"/>
         <geometry>
-          <mesh filename="package://snp_blending/meshes/mh180/visual/link_s.stl"/>
+          <mesh filename="package://snp_blending/urdf/mh180_120/visual/link_s.stl"/>
         </geometry>
         <material name="blue"/>
@@ -33,5 +33,5 @@
         <origin xyz="0 0 0" rpy="0 0 0"/>
         <geometry>
-          <mesh filename="package://snp_blending/meshes/mh180/collision/link_s.stl"/>
+          <mesh filename="package://snp_blending/urdf/mh180_120/collision/link_s.stl"/>
         </geometry>
         <material name="yellow"/>
@@ -42,5 +42,5 @@
         <origin xyz="0 0 0" rpy="0 0 0"/>
         <geometry>
-          <mesh filename="package://snp_blending/meshes/mh180/visual/link_l.stl"/>
+          <mesh filename="package://snp_blending/urdf/mh180_120/visual/link_l.stl"/>
         </geometry>
         <material name="blue"/>
@@ -49,5 +49,5 @@
         <origin xyz="0 0 0" rpy="0 0 0"/>
         <geometry>
-          <mesh filename="package://snp_blending/meshes/mh180/collision/link_l.stl"/>
+          <mesh filename="package://snp_blending/urdf/mh180_120/collision/link_l.stl"/>
         </geometry>
         <material name="yellow"/>
@@ -58,5 +58,5 @@
         <origin xyz="0 0 0" rpy="0 0 0"/>
         <geometry>
-          <mesh filename="package://snp_blending/meshes/mh180_120/visual/link_u.stl"/>
+          <mesh filename="package://snp_blending/urdf/mh180_120/visual/link_u.stl"/>
         </geometry>
         <material name="blue"/>
@@ -65,5 +65,5 @@
         <origin xyz="0 0 0" rpy="0 0 0"/>
         <geometry>
-          <mesh filename="package://snp_blending/meshes/mh180_120/collision/link_u.stl"/>
+          <mesh filename="package://snp_blending/urdf/mh180_120/collision/link_u.stl"/>
         </geometry>
         <material name="yellow"/>
@@ -74,5 +74,5 @@
         <origin xyz="0 0 0" rpy="0 0 0"/>
         <geometry>
-          <mesh filename="package://snp_blending/meshes/mh180_120/visual/link_r.stl"/>
+          <mesh filename="package://snp_blending/urdf/mh180_120/visual/link_r.stl"/>
         </geometry>
         <material name="blue"/>
@@ -81,5 +81,5 @@
         <origin xyz="0 0 0" rpy="0 0 0"/>
         <geometry>
-          <mesh filename="package://snp_blending/meshes/mh180_120/collision/link_r.stl"/>
+          <mesh filename="package://snp_blending/urdf/mh180_120/collision/link_r.stl"/>
         </geometry>
         <material name="yellow"/>
@@ -90,5 +90,5 @@
         <origin xyz="0 0 0" rpy="0 0 0"/>
         <geometry>
-          <mesh filename="package://snp_blending/meshes/mh180/visual/link_b.stl"/>
+          <mesh filename="package://snp_blending/urdf/mh180_120/visual/link_b.stl"/>
         </geometry>
         <material name="blue"/>
@@ -97,5 +97,5 @@
         <origin xyz="0 0 0" rpy="0 0 0"/>
         <geometry>
-          <mesh filename="package://snp_blending/meshes/mh180/collision/link_b.stl"/>
+          <mesh filename="package://snp_blending/urdf/mh180_120/collision/link_b.stl"/>
         </geometry>
         <material name="yellow"/>
@@ -106,5 +106,5 @@
         <origin xyz="0 0 0" rpy="0 0 0"/>
         <geometry>
-          <mesh filename="package://snp_blending/meshes/mh180/visual/link_t.stl"/>
+          <mesh filename="package://snp_blending/urdf/mh180_120/visual/link_t.stl"/>
         </geometry>
         <material name="black">
@@ -115,5 +115,5 @@
         <origin xyz="0 0 0" rpy="0 0 0"/>
         <geometry>
-          <mesh filename="package://snp_blending/meshes/mh180/collision/link_t.stl"/>
+          <mesh filename="package://snp_blending/urdf/mh180_120/collision/link_t.stl"/>
         </geometry>
         <material name="black"/>
