Commit message: Fix load_yaml difference between foxy and humble+

File: snp_automate_2022/urdf/workcell.xacro (robot description, xacro)
@@ -130,5 +130,11 @@
     <child link="ee"/>
   </joint>
-  <xacro:property name="camera_cal" value="${xacro.load_yaml('$(find snp_automate_2022)/config/camera_calibration.yaml')}" />
+  <xacro:arg name="ros_distro" default="humble"/>
+  <xacro:if value="${'$(arg ros_distro)' > 'foxy'}">
+    <xacro:property name="camera_cal" value="${xacro.load_yaml('$(find snp_automate_2022)/config/camera_calibration.yaml')}" />
+  </xacro:if>
+  <xacro:unless value="${'$(arg ros_distro)' > 'foxy'}">
+    <xacro:property name="camera_cal" value="${load_yaml('$(find snp_automate_2022)/config/camera_calibration.yaml')}" />
+  </xacro:unless>
   <link name="camera_color_optical_frame"/>
   <joint name="tool0_to_camera" type="fixed">
